File: spacebot-CM4-breakout.kicad_pcb (KiCad board)
At the start: 2 copper layers, 2 parts, among them J1 Conn_02x12_Counter_Clockwise, U1 Compute_Module_4_Connectors

Commit message: updates
Parts:
- added G***: LOGO, trylaarsdam:wcl_logo, F.Cu at (106.6, 74.3)
- moved J1 13.2 mm to (110.1, 111.4)
Connections:
- U1 pad 61: SD_DAT1 -> SD_DAT3
- U1 pad 63: SD_DAT2 -> SD_DAT0
- U1 pad 67: unconnected-(U1-Pad67) -> SD_DAT1
- U1 pad 69: unconnected-(U1-Pad69) -> SD_DAT2
Routing:
- net GND: track 0.00 -> 147.2 mm, vias 0 -> 19
- net 1.8V: track 0.00 -> 66.1 mm
- net SDA_0: track 0.00 -> 54.0 mm
- net I2S_SD: track 0.00 -> 53.5 mm, vias 0 -> 2
- net SCL_0: track 0.00 -> 51.7 mm
- net 3.3V: track 0.00 -> 37.4 mm, vias 0 -> 2
- net SD_CLK: track 0.00 -> 36.5 mm
- net I2S_WS: track 0.00 -> 35.2 mm, vias 0 -> 1
- net SD_DAT2: track 0.00 -> 28.8 mm, vias 0 -> 1
- net UART_RX: track 0.00 -> 28.6 mm, vias 0 -> 2
- net SD_DAT0: track 0.00 -> 28.5 mm
- net UART_TX: track 0.00 -> 27.3 mm, vias 0 -> 1
- net 5V: track 0.00 -> 25.7 mm
- net I2S_SCK: track 0.00 -> 25.5 mm, vias 0 -> 2
- net SD_DAT1: track 0.00 -> 25.1 mm, vias 0 -> 1
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- added copper zone on B.Cu, net GND
- added copper zone on F.Cu, net GND
Other:
- board outline added: 68 x 55.5 mm
- board text added: "1.8V"
- board text added: "3.3V"
- board text added: "5V"
- board text added: "GND"
- board text added: "I2S_SCK"
- board text added: "I2S_SD"
- board text added: "I2S_WS"
- board text added: "SCL0"
- board text added: "SDA0"
- board text added: "SD_CLK"
- board text added: "SD_DAT0"
- board text added: "SD_DAT1"
- board text added: "SD_DAT2"
- board text added: "SD_DAT3"
- board text added: "UART_RX"
- board text added: "UART_TX"
- board text added: "v1.0"

Commit message: updates
Parts:
- added D1: LED, LED_THT:LED_D3.0mm, F.Cu at (118.9, 121.6)
- J1: value Conn_02x12_Counter_Clockwise -> Conn_02x16_Counter_Clockwise; footprint Connector_PinHeader_2.54mm:PinHeader_2x12_P2.54mm_Horizontal -> Connector_PinHeader_2.54mm:PinHeader_2x16_P2.54mm_Horizontal
- moved J1 6.43 mm to (110.2, 117.8)
Connections:
- J1 pad 13: I2S_WS -> GPIO10
- J1 pad 14: SCL_0 -> GPIO27
- J1 pad 15: SDA_0 -> GPIO4
- J1 pad 16: unconnected-(J1-Pad16) -> GPIO2
- J1 pad 17: unconnected-(J1-Pad17) -> GPIO3
- J1 pad 18: unconnected-(J1-Pad18) -> GPIO17
- J1 pad 19: unconnected-(J1-Pad19) -> GPIO22
- J1 pad 20: unconnected-(J1-Pad20) -> GPIO9
- J1 pad 21: unconnected-(J1-Pad21) -> GPIO11
- J1 pad 22: GND -> GPIO5
- J1 pad 23: unconnected-(J1-Pad23) -> GPIO6
- J1 pad 24: 1.8V -> I2S_WS
- U1 pad 30: unconnected-(U1-Pad30) -> GPIO6
- U1 pad 34: unconnected-(U1-Pad34) -> GPIO5
- U1 pad 38: unconnected-(U1-Pad38) -> GPIO11
- U1 pad 40: unconnected-(U1-Pad40) -> GPIO9
- U1 pad 44: unconnected-(U1-Pad44) -> GPIO10
- U1 pad 46: unconnected-(U1-Pad46) -> GPIO22
- U1 pad 48: unconnected-(U1-Pad48) -> GPIO27
- U1 pad 50: unconnected-(U1-Pad50) -> GPIO17
- U1 pad 54: unconnected-(U1-Pad54) -> GPIO4
- U1 pad 56: unconnected-(U1-Pad56) -> GPIO3
- U1 pad 58: unconnected-(U1-Pad58) -> GPIO2
- U1 pad 89: unconnected-(U1-Pad89) -> WL_nDisable
- U1 pad 91: unconnected-(U1-Pad91) -> BT_nDisable
- U1 pad 93: unconnected-(U1-Pad93) -> nRPIBOOT
- U1 pad 95: unconnected-(U1-Pad95) -> Net-(U1-Pad95)
Routing:
- net WL_nDisable: track 0.00 -> 135.3 mm, vias 0 -> 1
- net BT_nDisable: track 0.00 -> 130.9 mm, vias 0 -> 1
- net nRPIBOOT: track 0.00 -> 122.3 mm, vias 0 -> 1
- net GPIO17: track 0.00 -> 75.4 mm, vias 0 -> 1
- net GPIO3: track 0.00 -> 74.9 mm, vias 0 -> 1
- net GPIO2: track 0.00 -> 71.5 mm, vias 0 -> 1
- net GPIO22: track 0.00 -> 71.0 mm, vias 0 -> 1
- net GPIO4: track 0.00 -> 68.0 mm, vias 0 -> 1
- net GPIO27: track 0.00 -> 63.5 mm, vias 0 -> 1
- net GPIO10: track 0.00 -> 56.8 mm, vias 0 -> 1
- net GPIO9: track 0.00 -> 56.6 mm, vias 0 -> 1
- net 1.8V: track 66.1 -> 121.0 mm, vias 0 -> 1
- net GPIO11: track 0.00 -> 49.5 mm, vias 0 -> 1
- net GPIO5: track 0.00 -> 45.7 mm, vias 0 -> 1
- net GPIO6: track 0.00 -> 38.6 mm
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Other:
- board text added: "v1.1"
- board text removed: "1.8V"
- board text removed: "3.3V"
- board text removed: "5V"
- board text removed: "GND"
- board text removed: "I2S_SCK"
- board text removed: "I2S_SD"
- board text removed: "I2S_WS"
- board text removed: "SCL0"
- board text removed: "SDA0"
- board text removed: "SD_CLK"
- board text removed: "SD_DAT0"
- board text removed: "SD_DAT1"
- board text removed: "SD_DAT2"
- board text removed: "SD_DAT3"
- board text removed: "UART_RX"
- board text removed: "UART_TX"
- board text removed: "v1.0"
